File: PCB/Schematico.sch (EAGLE design)
At the start: 18 parts, among them IC3 AT24CP

Commit message: PCB final
Parts:
- removed R3: (no value), adafruit:R-US_0204/7
- removed S2: (no value), switch:320-916
- added C4: 1uF, capacitor-wima:C2,5-3
- added C5: 4.7uF, capacitor-wima:C2,5-3
- added D1: 1N821, diode:1N821
- added IC1: (no value), v-reg:78XXS
- added J1: (no value), SparkFun-Connectors:CONN_02
- added JP5: (no value), adafruit:PINHD-1X6B
- added R1: 600k, adafruit:R-US_0204/7
- added R2: 1M, adafruit:R-US_0204/7
- added S3: (no value), SparkFun-Switches:SWITCH-SPDT-PTH-11.6X4.0MM
- added SV1: (no value), con-lstb:MA03-1
- C1: value (none) -> 0.1uF
- C2: value (none) -> 0.1u
- C3: value (none) -> 0.22uF
- R4, R5: value (none) -> 10k
Connections:
- new net BTLVL: JP2.2, R1.2, R2.1
- new net CTRL: JP2.8, SV1.2
- new net N$3: JP2.9, S1.2
- new net REF: JP2.6, SV1.3
- new net RX3V3: JP5.5, JP7.6
- new net RX5V: JP1.22, JP8.6
- new net TX3V3: JP5.4, JP7.5
- new net TX5V: JP1.23, JP8.5
- new net VBAT: C3.1, IC2.IN, R1.1, S3.O
- new net WRK: JP2.16, SV1.1
- net 3V3: now also C4.1, IC1.OUT; no longer C1.1, IC2.OUT
- net 5V: now also C1.1, C5.1, D1.C, IC1.IN, IC2.OUT, JP1.1, JP3.1, JP5.2, R4.2, R5.2; no longer C3.1, IC2.IN
- net GND: now also C2.2, C4.2, C5.2, D1.A, IC1.GND, J1.2, JP1.2, JP4.1, JP5.3, R2.2, S1.1
- net N$1: now also J1.1, S3.P; no longer IC3.SCL, R5.1
- net N$2: now also C2.1, JP2.3; no longer IC3.SDA, R4.1
- net SCL5V: now also IC3.SCL, JP1.11, R5.1; no longer R5.2
- net SDA5V: now also IC3.SDA, JP1.12, R4.1; no longer R4.2
Other:
- note added: "3.3V Voltage regulator"
- note added: "5V Voltage regulator"
- note added: "Battery Power Supply"
- note added: "Battery level monitor"
- note added: "Bluetooth module"
- note added: "Ceramic"
- note added: "ELECTRONIC TECHNOLOGIES AND BIOSENSORS LABORATORY Authors: Group 2"
- note added: "Glucose strip"
- note added: "Note: UART TX and RX channels are named with respect to HC05 Bluetooth module"
- note added: "PSoC5 Kit"
- note removed: "Voltage regulator"
- moved on the sheet: C1, C2, C3, IC3, JP1, JP2, JP3, JP4, JP9, R4, R5, S1
